File: Kicad/RPi_CAN_BUS.sch (KiCad schematic (older format))
At the start: 7 parts, among them U4 MCP25625, Y1 16MHz

Commit message: Mise a jour du 6 juillet 2017
Parts:
- added R6: 10k, Resistors_SMD:R_0805_HandSoldering, symbol R
Connections:
- net +3V3: now also R6.1
- net GND: now also U4.5 (STBY)
- net at U4.18 (~RESET): now also R6.2
- no-connect marks 8 -> 6
Changed lines of the file:
@@
 $EndComp
 $Comp
-L GND #PWR037
+L GND #PWR030
 U 1 1 589B5818
 P 3900 5300
-F 0 "#PWR037" H 3950 5350 50  0001 C CNN
+F 0 "#PWR030" H 3950 5350 50  0001 C CNN
 F 1 "GND" H 3905 5127 50  0000 C CNN
 F 2 "" H -1550 125 50  0001 C CNN
@@
 $EndComp
 $Comp
-L GND #PWR038
+L GND #PWR031
 U 1 1 589B581E
 P 4200 5300
-F 0 "#PWR038" H 4250 5350 50  0001 C CNN
+F 0 "#PWR031" H 4250 5350 50  0001 C CNN
 F 1 "GND" H 4205 5127 50  0000 C CNN
 F 2 "" H -1550 125 50  0001 C CNN
@@
 $EndComp
 NoConn ~ 3400 4575
-NoConn ~ 3400 4475
 NoConn ~ 3400 4375
 NoConn ~ 3400 4275
@@
 $EndComp
 $Comp
-L GND #PWR039
+L GND #PWR032
 U 1 1 589B5839
 P 3375 2050
-F 0 "#PWR039" H -1550 -125 50  0001 C CNN
+F 0 "#PWR032" H -1550 -125 50  0001 C CNN
 F 1 "GND" H 3380 1877 50  0000 C CNN
 F 2 "" H -1550 125 50  0001 C CNN
@@
 	3550 2400 3375 2400
 $Comp
-L GND #PWR040
+L GND #PWR033
 U 1 1 589B5850
 P 3375 2400
-F 0 "#PWR040" H -1550 -125 50  0001 C CNN
+F 0 "#PWR033" H -1550 -125 50  0001 C CNN
 F 1 "GND" H 3380 2227 50  0000 C CNN
 F 2 "" H -1550 125 50  0001 C CNN
@@
 $EndComp
 $Comp
-L +3.3V #PWR041
+L +3.3V #PWR034
 U 1 1 589B5856
 P 4050 1875
-F 0 "#PWR041" H -1550 -25 50  0001 C CNN
+F 0 "#PWR034" H -1550 -25 50  0001 C CNN
 F 1 "+3.3V" H 4065 2048 50  0000 C CNN
 F 2 "" H -1550 125 50  0001 C CNN
@@
 	4250 1875 4250 2475
 $Comp
-L +5V #PWR042
+L +5V #PWR035
 U 1 1 589B585D
 P 4250 1875
-F 0 "#PWR042" H -1550 -50 50  0001 C CNN
+F 0 "#PWR035" H -1550 -50 50  0001 C CNN
 F 1 "+5V" H 4265 2048 50  0000 C CNN
 F 2 "" H -1550 100 50  0001 C CNN
@@
 	4625 2400 4800 2400
 $Comp
-L GND #PWR043
+L GND #PWR036
 U 1 1 589B586D
 P 4800 2400
-F 0 "#PWR043" H -1550 -125 50  0001 C CNN
+F 0 "#PWR036" H -1550 -125 50  0001 C CNN
 F 1 "GND" H 4805 2227 50  0000 C CNN
 F 2 "" H -1550 125 50  0001 C CNN
@@
 	1    0    0    -1
 $EndComp
-NoConn ~ 3400 3375
 $Comp
 L C_Small C4
@@
 Connection ~ 5450 4575
 $Comp
-L GND #PWR044
+L GND #PWR037
 U 1 1 589B5898
 P 5450 4775
-F 0 "#PWR044" H 5500 4825 50  0001 C CNN
+F 0 "#PWR037" H 5500 4825 50  0001 C CNN
 F 1 "GND" H 5455 4602 50  0000 C CNN
 F 2 "" H 0   -400 50  0001 C CNN
@@
 Text HLabel 3400 3875 0    60   Output ~ 0
 ~INT
+Wire Wire Line
+	3400 3375 2950 3375
+Wire Wire Line
+	2950 3375 2950 3425
+$Comp
+L GND #PWR038
+U 1 1 5935FEFC
+P 2950 3425
+F 0 "#PWR038" H -1975 900 50  0001 C CNN
+F 1 "GND" H 2955 3252 50  0000 C CNN
+F 2 "" H -1975 1150 50  0001 C CNN
+F 3 "" H -1975 1150 50  0001 C CNN
+	1    2950 3425
+	1    0    0    -1
+$EndComp
+Wire Wire Line
+	3400 4475 2625 4475
+Wire Wire Line
+	2625 4475 2625 4300
+$Comp
+L R R6
+U 1 1 5935FFC7
+P 2625 4150
+F 0 "R6" H 2695 4196 50  0000 L CNN
+F 1 "10k" H 2695 4105 50  0000 L CNN
+F 2 "Resistors_SMD:R_0805_HandSoldering" V 2555 4150 50  0001 C CNN
+F 3 "" H 2625 4150 50  0001 C CNN
+	1    2625 4150
+	1    0    0    -1
+$EndComp
+$Comp
+L +3.3V #PWR039
+U 1 1 59360100
+P 2625 3925
+F 0 "#PWR039" H -2975 2025 50  0001 C CNN
+F 1 "+3.3V" H 2640 4098 50  0000 C CNN
+F 2 "" H -2975 2175 50  0001 C CNN
+F 3 "" H -2975 2175 50  0001 C CNN
+	1    2625 3925
+	1    0    0    -1
+$EndComp
+Wire Wire Line
+	2625 3925 2625 4000
 $EndSCHEMATC
