File: Kicad/RPi_Hat.kicad_pcb (KiCad board)
At the start: 2 copper layers, 65 x 56.5 mm, 44 parts, among them J1 RPi_GPIO, J4 CAN_NODE_JUNCTION, J5 CAN_NODE_JUNCTION, U1 DS3231, U4 MCP25625, U5 MCP25625, U6 PCA9306, U7 DS2482-100, U8 DS9503, Y1 16MHz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

Commit message: Mise a jour du 6 juillet 2017
Parts:
- added C16: 1uF, Capacitors_SMD:C_0805_HandSoldering, B.Cu at (146.6, 101.7)
- added R6: 10k, Resistors_SMD:R_0805_HandSoldering, B.Cu at (107.6, 80.9)
- added R7: 10k, Resistors_SMD:R_0805_HandSoldering, B.Cu at (106.9, 105.7)
- moved C4 0.32 mm to (98.1, 76.1)
- moved C5 0.32 mm to (98.1, 83.4)
Connections:
- Adafruit_Feather-1 pad 24: /feather_connectors/D9 -> /RTC/INT_SQW
- Adafruit_Feather_Wing-1 pad 24: /feather_connectors/D9 -> /RTC/INT_SQW
- U1 pad 3: Net-(U1-Pad3) -> /RTC/INT_SQW
- U4 pad 5: Net-(U4-Pad5) -> GND
- U5 pad 5: Net-(U5-Pad5) -> GND
Routing:
- net /RTC/INT_SQW: track 0.00 -> 45.9 mm, vias 0 -> 1
- net /feather_connectors/D9: track 32.4 -> 0.00 mm
- net Net-(R7-Pad2): track 0.00 -> 3.93 mm, vias 0 -> 1
- net /feather_connectors/FEATHER_3.3V: track 130.5 -> 134.2 mm, vias 3 -> 4
- net Net-(R6-Pad2): track 0.00 -> 3.56 mm, vias 0 -> 1
- net +3V3: track 113.8 -> 116.7 mm, vias 3 -> 4
- net +5V: track 172.9 -> 170.3 mm
- net /1-wire/1_WIRE_GND: track 10.7 -> 12.6 mm, vias 0 -> 1
- net GND: track 419.2 -> 420.9 mm
- net /RPi_GPIO/swdio: track 40.5 -> 41.9 mm
- net /CAN-: track 92.0 -> 92.8 mm
- net /RPi_GPIO/RPi_MOSI_SPI: track 29.5 -> 30.2 mm
- net /RPi_GPIO/RPi_SDA_I2C: track 67.5 -> 68.2 mm
- net /RPi_GPIO/RPi_SCL_I2C: track 69.4 -> 70.1 mm
Other:
- board text added: "3V3"
- board text added: "5V"
- board text added: "CANH"
- board text added: "CANL"
- board text added: "Cob St-Ambroise RPi Hat Feather V. 1.1 Juin 2017"
- board text added: "GND"
- board text added: "IO"
- board text added: "SCL"
- board text added: "SDA"
- board text removed: "Cob St-Ambroise RPi Hat Feather V. 1.0 Avril 2017"
