File: Kicad/RPi_Hat.sch (KiCad schematic (older format))
At the start: 7 parts, among them J4 CAN_NODE_JUNCTION, J5 CAN_NODE_JUNCTION

Commit message: Mise a jour du 6 juillet 2017
Parts:
- added C16: 1uF, Capacitors_SMD:C_0805_HandSoldering, symbol C_Small
Connections:
- net +5V: now also C16.2
- net 1-wire/1_WIRE_GND: now also C16.1
Other:
- moved on the sheet: 1Wire-1
Changed lines of the file:
@@
 $EndSheet
+$Sheet
+S 1800 1850 1275 625
+U 58965077
+F0 "1-wire" 60
+F1 "1-wire.sch" 60
+F2 "SCL" I R 3075 2075 60
+F3 "SDA" B R 3075 1975 60
+F4 "1_WIRE_IO" B L 1800 2175 60
+F5 "1_WIRE_GND" U L 1800 2275 60
+$EndSheet
+$Sheet
+S 5325 2850 1700 825
+U 589B5416
+F0 "RPi_CAN_BUS" 60
+F1 "RPi_CAN_BUS.sch" 60
+F2 "~CS" I L 5325 3375 60
+F3 "SCK" I L 5325 3250 60
+F4 "SI" I L 5325 3000 60
+F5 "SO" O L 5325 3125 60
+F6 "CANH" B R 7025 3075 60
+F7 "CANL" B R 7025 3175 60
+F8 "~INT" O L 5325 3500 60
+$EndSheet
+$Sheet
+S 7450 1625 1025 925
+U 589B5AEE
+F0 "feather_CAN_BUS" 60
+F1 "feather_CAN_BUS.sch" 60
+F2 "~CS" I L 7450 2250 60
+F3 "SCK" I L 7450 2125 60
+F4 "SI" I L 7450 1875 60
+F5 "SO" O L 7450 2000 60
+F6 "~INT" O L 7450 2375 60
+F7 "CANH" B R 8475 2150 60
+F8 "CANL" B R 8475 2250 60
+F9 "V_IO" U L 7450 1750 60
+$EndSheet
+$Comp
+L CONN_01X02 CAN1
+U 1 1 589BA6CF
+P 9425 1750
+F 0 "CAN1" H 9503 1791 50  0000 L CNN
+F 1 "CONN_01X02" H 9503 1700 50  0000 L CNN
+F 2 "caribou:0436500219" H 8125 -650 50  0001 C CNN
+F 3 "" H 8125 -650 50  0001 C CNN
+	1    9425 1750
+	1    0    0    -1
+$EndComp
+$Comp
+L CONN_01X02 CAN2
+U 1 1 589BA6D6
+P 9450 3925
+F 0 "CAN2" H 9528 3966 50  0000 L CNN
+F 1 "CONN_01X02" H 9528 3875 50  0000 L CNN
+F 2 "caribou:0436500219" H 8150 1525 50  0001 C CNN
+F 3 "" H 8150 1525 50  0001 C CNN
+	1    9450 3925
+	1    0    0    -1
+$EndComp
+Text Label 9000 2675 2    60   ~ 0
+CAN+
+Text Label 9100 2675 0    60   ~ 0
+CAN-
+$Comp
+L CONN_01X04 I2C-1
+U 1 1 589E2857
+P 9425 1325
+F 0 "I2C-1" H 9503 1366 50  0000 L CNN
+F 1 "CONN_01X04" H 9503 1275 50  0000 L CNN
+F 2 "caribou:0436500417" H 175 -375 50  0001 C CNN
+F 3 "" H 175 -375 50  0001 C CNN
+	1    9425 1325
+	1    0    0    -1
+$EndComp
+$Comp
+L GND #PWR01
+U 1 1 589E2862
+P 9075 1100
+F 0 "#PWR01" H 9075 850 50  0001 C CNN
+F 1 "GND" H 9075 950 50  0000 C CNN
+F 2 "" H 9075 1100 50  0000 C CNN
+F 3 "" H 9075 1100 50  0000 C CNN
+	1    9075 1100
+	-1   0    0    1
+$EndComp
+$Comp
+L CONN_01X03 1Wire-1
+U 1 1 58A1C4EE
+P 1125 2175
+F 0 "1Wire-1" H 1203 2216 50  0000 L CNN
+F 1 "CONN_01X03" H 1203 2125 50  0000 L CNN
+F 2 "caribou:0436500317" H -4650 -2925 50  0001 C CNN
+F 3 "" H -4650 -2925 50  0001 C CNN
+	1    1125 2175
+	-1   0    0    1
+$EndComp
+$Comp
+L +5V #PWR02
+U 1 1 58A1C4F5
+P 1675 2025
+F 0 "#PWR02" H 75  -2075 50  0001 C CNN
+F 1 "+5V" H 1690 2198 50  0000 C CNN
+F 2 "" H 75  -1925 50  0001 C CNN
+F 3 "" H 75  -1925 50  0001 C CNN
+	1    1675 2025
+	-1   0    0    -1
+$EndComp
+$Comp
+L CAN_NODE_JUNCTION J5
+U 1 1 58AA1A82
+P 8975 2200
+F 0 "J5" H 9203 2246 50  0000 L CNN
+F 1 "CAN_NODE_JUNCTION" H 9203 2155 50  0000 L CNN
+F 2 "caribou:CAN_NODE_JONCTION" H -800 -1225 50  0001 C CNN
+F 3 "" H -800 -1225 50  0001 C CNN
+	1    8975 2200
+	1    0    0    -1
+$EndComp
+$Comp
+L CAN_NODE_JUNCTION J4
+U 1 1 58AB23E0
+P 8975 3125
+F 0 "J4" H 9203 3171 50  0000 L CNN
+F 1 "CAN_NODE_JUNCTION" H 9203 3080 50  0000 L CNN
+F 2 "caribou:CAN_NODE_JONCTION" H -800 -300 50  0001 C CNN
+F 3 "" H -800 -300 50  0001 C CNN
+	1    8975 3125
+	1    0    0    -1
+$EndComp
+Text Label 8775 2150 2    60   ~ 0
+CAN+
+Text Label 8525 2250 0    60   ~ 0
+CAN-
+Text Label 7975 3075 2    60   ~ 0
+CAN+
+Text Label 7725 3175 0    60   ~ 0
+CAN-
+Text Label 9100 3575 0    60   ~ 0
+CAN-
+Text Label 9000 3575 2    60   ~ 0
+CAN+
+Text Label 9100 1900 0    60   ~ 0
+CAN-
+Text Label 9000 1900 2    60   ~ 0
+CAN+
+$Comp
+L C_Small C15
+U 1 1 590057AA
+P 8500 950
+F 0 "C15" V 8271 950 50  0000 C CNN
+F 1 "0.1u" V 8362 950 50  0000 C CNN
+F 2 "Capacitors_SMD:C_0805_HandSoldering" H 3250 -1125 50  0001 C CNN
+F 3 "" H 3250 -1125 50  0001 C CNN
+	1    8500 950
+	0    1    1    0
+$EndComp
+$Comp
+L GND #PWR03
+U 1 1 59008424
+P 8700 1025
+F 0 "#PWR03" H 8700 775 50  0001 C CNN
+F 1 "GND" H 8705 852 50  0000 C CNN
+F 2 "" H 8700 1025 50  0001 C CNN
+F 3 "" H 8700 1025 50  0001 C CNN
+	1    8700 1025
+	1    0    0    -1
+$EndComp
 $Sheet
 S 1800 1050 1275 600
@@
 F2 "SCL" I R 3075 1475 60
 F3 "SDA" B R 3075 1375 60
+F4 "INT_SQW" O L 1800 1175 60
 $EndSheet
 $Sheet
@@
 F13 "FEATHER_MISO_SPI" I R 7025 2000 60
 F14 "FEATHER_3.3V" U R 7025 1275 60
-$EndSheet
-$Sheet
-S 1800 1850 1275 625
-U 58965077
-F0 "1-wire" 60
-F1 "1-wire.sch" 60
-F2 "SCL" I R 3075 2075 60
-F3 "SDA" B R 3075 1975 60
-F4 "1_WIRE_IO" B L 1800 2175 60
-F5 "1_WIRE_GND" U L 1800 2275 60
-$EndSheet
-$Sheet
-S 5325 2850 1700 825
-U 589B5416
-F0 "RPi_CAN_BUS" 60
-F1 "RPi_CAN_BUS.sch" 60
-F2 "~CS" I L 5325 3375 60
-F3 "SCK" I L 5325 3250 60
-F4 "SI" I L 5325 3000 60
-F5 "SO" O L 5325 3125 60
-F6 "CANH" B R 7025 3075 60
-F7 "CANL" B R 7025 3175 60
-F8 "~INT" O L 5325 3500 60
-$EndSheet
-$Sheet
-S 7450 1625 1025 925
-U 589B5AEE
-F0 "feather_CAN_BUS" 60
-F1 "feather_CAN_BUS.sch" 60
-F2 "~CS" I L 7450 2250 60
-F3 "SCK" I L 7450 2125 60
-F4 "SI" I L 7450 1875 60
-F5 "SO" O L 7450 2000 60
-F6 "~INT" O L 7450 2375 60
-F7 "CANH" B R 8475 2150 60
-F8 "CANL" B R 8475 2250 60
-F9 "V_IO" U L 7450 1750 60
-$EndSheet
-$Comp
-L CONN_01X02 CAN1
-U 1 1 589BA6CF
-P 9425 1750
-F 0 "CAN1" H 9503 1791 50  0000 L CNN
-F 1 "CONN_01X02" H 9503 1700 50  0000 L CNN
-F 2 "caribou:0436500219" H 8125 -650 50  0001 C CNN
-F 3 "" H 8125 -650 50  0001 C CNN
-	1    9425 1750
-	1    0    0    -1
-$EndComp
-$Comp
-L CONN_01X02 CAN2
-U 1 1 589BA6D6
-P 9450 3925
-F 0 "CAN2" H 9528 3966 50  0000 L CNN
-F 1 "CONN_01X02" H 9528 3875 50  0000 L CNN
-F 2 "caribou:0436500219" H 8150 1525 50  0001 C CNN
-F 3 "" H 8150 1525 50  0001 C CNN
-	1    9450 3925
-	1    0    0    -1
-$EndComp
-Text Label 9000 2675 2    60   ~ 0
-CAN+
-Text Label 9100 2675 0    60   ~ 0
-CAN-
-$Comp
-L CONN_01X04 I2C-1
-U 1 1 589E2857
-P 9425 1325
-F 0 "I2C-1" H 9503 1366 50  0000 L CNN
-F 1 "CONN_01X04" H 9503 1275 50  0000 L CNN
-F 2 "caribou:0436500417" H 175 -375 50  0001 C CNN
-F 3 "" H 175 -375 50  0001 C CNN
-	1    9425 1325
-	1    0    0    -1
-$EndComp
-$Comp
-L GND #PWR01
-U 1 1 589E2862
-P 9075 1100
-F 0 "#PWR01" H 9075 850 50  0001 C CNN
-F 1 "GND" H 9075 950 50  0000 C CNN
-F 2 "" H 9075 1100 50  0000 C CNN
-F 3 "" H 9075 1100 50  0000 C CNN
-	1    9075 1100
-	-1   0    0    1
-$EndComp
-$Comp
-L CONN_01X03 1Wire-1
-U 1 1 58A1C4EE
-P 1475 2175
-F 0 "1Wire-1" H 1553 2216 50  0000 L CNN
-F 1 "CONN_01X03" H 1553 2125 50  0000 L CNN
-F 2 "caribou:0436500317" H -4300 -2925 50  0001 C CNN
-F 3 "" H -4300 -2925 50  0001 C CNN
-	1    1475 2175
-	-1   0    0    1
-$EndComp
-$Comp
-L +5V #PWR02
-U 1 1 58A1C4F5
-P 1675 2025
-F 0 "#PWR02" H 75  -2075 50  0001 C CNN
-F 1 "+5V" H 1690 2198 50  0000 C CNN
-F 2 "" H 75  -1925 50  0001 C CNN
-F 3 "" H 75  -1925 50  0001 C CNN
-	1    1675 2025
-	-1   0    0    -1
-$EndComp
-$Comp
-L CAN_NODE_JUNCTION J5
-U 1 1 58AA1A82
-P 8975 2200
-F 0 "J5" H 9203 2246 50  0000 L CNN
-F 1 "CAN_NODE_JUNCTION" H 9203 2155 50  0000 L CNN
-F 2 "caribou:CAN_NODE_JONCTION" H -800 -1225 50  0001 C CNN
-F 3 "" H -800 -1225 50  0001 C CNN
-	1    8975 2200
-	1    0    0    -1
-$EndComp
-$Comp
-L CAN_NODE_JUNCTION J4
-U 1 1 58AB23E0
-P 8975 3125
-F 0 "J4" H 9203 3171 50  0000 L CNN
-F 1 "CAN_NODE_JUNCTION" H 9203 3080 50  0000 L CNN
-F 2 "caribou:CAN_NODE_JONCTION" H -800 -300 50  0001 C CNN
-F 3 "" H -800 -300 50  0001 C CNN
-	1    8975 3125
-	1    0    0    -1
-$EndComp
-Text Label 8775 2150 2    60   ~ 0
-CAN+
-Text Label 8525 2250 0    60   ~ 0
-CAN-
-Text Label 7975 3075 2    60   ~ 0
-CAN+
-Text Label 7725 3175 0    60   ~ 0
-CAN-
-Text Label 9100 3575 0    60   ~ 0
-CAN-
-Text Label 9000 3575 2    60   ~ 0
-CAN+
-Text Label 9100 1900 0    60   ~ 0
-CAN-
-Text Label 9000 1900 2    60   ~ 0
-CAN+
-$Comp
-L C_Small C15
-U 1 1 590057AA
-P 8500 950
-F 0 "C15" V 8271 950 50  0000 C CNN
-F 1 "0.1u" V 8362 950 50  0000 C CNN
-F 2 "Capacitors_SMD:C_0805_HandSoldering" H 3250 -1125 50  0001 C CNN
-F 3 "" H 3250 -1125 50  0001 C CNN
-	1    8500 950
-	0    1    1    0
+F15 "INT_SQW" I R 7025 1175 60
+$EndSheet
+$Comp
+L C_Small C16
+U 1 1 5936FEF7
+P 1525 2500
+F 0 "C16" V 1400 2500 50  0000 C CNN
+F 1 "1uF" V 1650 2500 50  0000 C CNN
+F 2 "Capacitors_SMD:C_0805_HandSoldering" H 1525 2500 50  0001 C CNN
+F 3 "" H 1525 2500 50  0001 C CNN
+	1    1525 2500
+	0    -1   -1   0
 $EndComp
 Wire Wire Line
@@
 Connection ~ 3175 1375
 Wire Wire Line
-	1675 2025 1675 2075
-Wire Wire Line
 	7025 1275 9225 1275
 Wire Wire Line
@@
 	9100 2500 9100 2825
 Wire Wire Line
-	1675 2175 1800 2175
-Wire Wire Line
-	1675 2275 1800 2275
+	1325 2175 1800 2175
+Wire Wire Line
+	1325 2275 1800 2275
 Wire Wire Line
 	8600 950  8700 950
 Wire Wire Line
 	8700 950  8700 1025
-$Comp
-L GND #PWR03
-U 1 1 59008424
-P 8700 1025
-F 0 "#PWR03" H 8700 775 50  0001 C CNN
-F 1 "GND" H 8705 852 50  0000 C CNN
-F 2 "" H 8700 1025 50  0001 C CNN
-F 3 "" H 8700 1025 50  0001 C CNN
-	1    8700 1025
-	1    0    0    -1
-$EndComp
 Wire Wire Line
 	8400 950  8275 950
@@
 	8275 950  8275 1275
 Connection ~ 8275 1275
+Wire Wire Line
+	1800 1175 1625 1175
+Wire Wire Line
+	1625 1175 1625 750
+Wire Wire Line
+	1625 750  7325 750
+Wire Wire Line
+	7325 750  7325 1175
+Wire Wire Line
+	7325 1175 7025 1175
+Wire Wire Line
+	1325 2075 1675 2075
+Wire Wire Line
+	1675 2025 1675 2500
+Connection ~ 1675 2075
+Wire Wire Line
+	1675 2500 1625 2500
+Wire Wire Line
+	1425 2500 1375 2500
+Wire Wire Line
+	1375 2500 1375 2275
+Connection ~ 1375 2275
 $EndSCHEMATC
