File: Kicad/feather_CAN_BUS.sch (KiCad schematic (older format))
At the start: 7 parts, among them U5 MCP25625, Y2 16MHz

Commit message: Mise a jour du 6 juillet 2017
Parts:
- added R7: 10k, Resistors_SMD:R_0805_HandSoldering, symbol R
Connections:
- net GND: now also U5.5 (STBY)
- net V_IO: now also R7.1
- net at U5.18 (~RESET): now also R7.2
- no-connect marks 8 -> 6
Changed lines of the file:
@@
 $EndComp
 $Comp
-L GND #PWR045
+L GND #PWR040
 U 1 1 589B70FD
 P 4975 5325
-F 0 "#PWR045" H 5025 5375 50  0001 C CNN
+F 0 "#PWR040" H 5025 5375 50  0001 C CNN
 F 1 "GND" H 4980 5152 50  0000 C CNN
 F 2 "" H -475 150 50  0001 C CNN
@@
 $EndComp
 $Comp
-L GND #PWR046
+L GND #PWR041
 U 1 1 589B7103
 P 5275 5325
-F 0 "#PWR046" H 5325 5375 50  0001 C CNN
+F 0 "#PWR041" H 5325 5375 50  0001 C CNN
 F 1 "GND" H 5280 5152 50  0000 C CNN
 F 2 "" H -475 150 50  0001 C CNN
@@
 $EndComp
 NoConn ~ 4475 4600
-NoConn ~ 4475 4500
 NoConn ~ 4475 4400
 NoConn ~ 4475 4300
@@
 $EndComp
 $Comp
-L GND #PWR047
+L GND #PWR042
 U 1 1 589B711E
 P 4450 2075
-F 0 "#PWR047" H -475 -100 50  0001 C CNN
+F 0 "#PWR042" H -475 -100 50  0001 C CNN
 F 1 "GND" H 4455 1902 50  0000 C CNN
 F 2 "" H -475 150 50  0001 C CNN
@@
 	4625 2425 4450 2425
 $Comp
-L GND #PWR048
+L GND #PWR043
 U 1 1 589B7135
 P 4450 2425
-F 0 "#PWR048" H -475 -100 50  0001 C CNN
+F 0 "#PWR043" H -475 -100 50  0001 C CNN
 F 1 "GND" H 4455 2252 50  0000 C CNN
 F 2 "" H -475 150 50  0001 C CNN
@@
 	5325 1900 5325 2500
 $Comp
-L +5V #PWR049
+L +5V #PWR044
 U 1 1 589B713C
 P 5325 1900
-F 0 "#PWR049" H -475 -25 50  0001 C CNN
+F 0 "#PWR044" H -475 -25 50  0001 C CNN
 F 1 "+5V" H 5340 2073 50  0000 C CNN
 F 2 "" H -475 125 50  0001 C CNN
@@
 	5700 2425 5875 2425
 $Comp
-L GND #PWR050
+L GND #PWR045
 U 1 1 589B714C
 P 5875 2425
-F 0 "#PWR050" H -475 -100 50  0001 C CNN
+F 0 "#PWR045" H -475 -100 50  0001 C CNN
 F 1 "GND" H 5880 2252 50  0000 C CNN
 F 2 "" H -475 150 50  0001 C CNN
@@
 	1    0    0    -1
 $EndComp
-NoConn ~ 4475 3400
 Wire Wire Line
 	5125 1625 5075 1625
@@
 Connection ~ 6550 4600
 $Comp
-L GND #PWR051
+L GND #PWR046
 U 1 1 589B7179
 P 6550 4800
-F 0 "#PWR051" H 6600 4850 50  0001 C CNN
+F 0 "#PWR046" H 6600 4850 50  0001 C CNN
 F 1 "GND" H 6555 4627 50  0000 C CNN
 F 2 "" H 1100 -375 50  0001 C CNN
@@
 Text HLabel 5075 1625 0    60   UnSpc ~ 0
 V_IO
+Wire Wire Line
+	4475 3400 4150 3400
+Wire Wire Line
+	4150 3400 4150 3575
+$Comp
+L GND #PWR047
+U 1 1 59360E26
+P 4150 3575
+F 0 "#PWR047" H -775 1050 50  0001 C CNN
+F 1 "GND" H 4155 3402 50  0000 C CNN
+F 2 "" H -775 1300 50  0001 C CNN
+F 3 "" H -775 1300 50  0001 C CNN
+	1    4150 3575
+	1    0    0    -1
+$EndComp
+Wire Wire Line
+	4475 4500 4000 4500
+Wire Wire Line
+	4000 4500 4000 4400
+$Comp
+L R R7
+U 1 1 59360F9A
+P 4000 4250
+F 0 "R7" H 4070 4296 50  0000 L CNN
+F 1 "10k" H 4070 4205 50  0000 L CNN
+F 2 "Resistors_SMD:R_0805_HandSoldering" V 3930 4250 50  0001 C CNN
+F 3 "" H 4000 4250 50  0001 C CNN
+	1    4000 4250
+	1    0    0    -1
+$EndComp
+Text HLabel 3925 4000 0    60   UnSpc ~ 0
+V_IO
+Wire Wire Line
+	4000 4100 4000 4000
+Wire Wire Line
+	4000 4000 3925 4000
 $EndSCHEMATC
