File: Kicad/feather_connector.sch (KiCad schematic (older format))
At the start: 2 parts

Commit message: Mise a jour du 6 juillet 2017
Parts:
- Adafruit_Feather-1: symbol FEATHER_MO_LORA-RESCUE-pihat_template -> FEATHER_MO_LORA
Connections:
- net labels added: INT_SQW
Changed lines of the file:
@@
 $Descr USLetter 11000 8500
 encoding utf-8
-Sheet 4 7
+Sheet 7 7
 Title ""
 Date "2017-02-08"
@@
 $EndDescr
 $Comp
-L FEATHER_MO_LORA-RESCUE-pihat_template Adafruit_Feather-1
+L FEATHER_MO_LORA Adafruit_Feather-1
 U 1 1 587BD5DB
 P 4275 3725
-F 0 "Adafruit_Feather-1" H 4725 2450 60  0000 C CNN
+F 0 "Adafruit_Feather-1" H 5000 2450 60  0000 C CNN
 F 1 "FEATHER_MO_LORA" H 4225 4875 60  0000 C CNN
 F 2 "caribou:FEATHER_MO_LORA" H 4275 4200 60  0001 C CNN
@@
 $EndComp
 $Comp
-L GND #PWR024
+L GND #PWR052
 U 1 1 587BD966
 P 2750 3250
-F 0 "#PWR024" H 2750 3000 50  0001 C CNN
+F 0 "#PWR052" H 2750 3000 50  0001 C CNN
 F 1 "GND" H 2750 3100 50  0000 C CNN
 F 2 "" H 2750 3250 50  0000 C CNN
@@
 SDA
 $Comp
-L GND #PWR025
+L GND #PWR053
 U 1 1 587C072D
 P 5900 3225
-F 0 "#PWR025" H 5900 2975 50  0001 C CNN
+F 0 "#PWR053" H 5900 2975 50  0001 C CNN
 F 1 "GND" H 5900 3075 50  0000 C CNN
 F 2 "" H 5900 3225 50  0000 C CNN
@@
 NoConn ~ 6725 4500
 $Comp
-L +5V #PWR026
+L +5V #PWR054
 U 1 1 589285EE
 P 5475 3525
-F 0 "#PWR026" H 150 -225 50  0001 C CNN
+F 0 "#PWR054" H 150 -225 50  0001 C CNN
 F 1 "+5V" H 5490 3698 50  0000 C CNN
 F 2 "" H 150 -75 50  0001 C CNN
@@
 	8650 3500 8650 3350
 $Comp
-L +5V #PWR027
+L +5V #PWR055
 U 1 1 58928823
 P 8650 3350
-F 0 "#PWR027" H 8700 3400 50  0001 C CNN
+F 0 "#PWR055" H 8700 3400 50  0001 C CNN
 F 1 "+5V" H 8665 3523 50  0000 C CNN
 F 2 "" H 0   0   50  0001 C CNN
@@
 Text HLabel 2925 2950 0    60   UnSpc ~ 0
 FEATHER_3.3V
+Text HLabel 5275 4200 2    60   Input ~ 0
+INT_SQW
 $EndSCHEMATC
