File: Kicad/1-wire.sch (KiCad schematic (older format))
At the start: 9 parts, among them U6 PCA9306, U7 DS2482-100, U8 DS9503

Commit message: Reouverture avec une nouvelle version de Kicad
Parts:
- C11, C12: symbol C -> RPi_Hat-rescue:C-RESCUE-RPi_Hat
- C13: symbol C_Small -> RPi_Hat-rescue:C_Small-RESCUE-RPi_Hat
- R1, R2, R3: symbol R -> RPi_Hat-rescue:R-RESCUE-RPi_Hat
- U6: symbol PCA9306-RESCUE-RPi_Hat -> RPi_Hat-rescue:PCA9306-RESCUE-RPi_Hat
- U7: symbol DS2482-100 -> jfng:DS2482-100
- U8: symbol DS9503 -> jfng:DS9503
Changed lines of the file:
@@
-EESchema Schematic File Version 2
-LIBS:RPi_Hat-rescue
-LIBS:power
-LIBS:device
-LIBS:transistors
-LIBS:conn
-LIBS:linear
-LIBS:regul
-LIBS:74xx
-LIBS:cmos4000
-LIBS:adc-dac
-LIBS:memory
-LIBS:xilinx
-LIBS:microcontrollers
-LIBS:dsp
-LIBS:microchip
-LIBS:analog_switches
-LIBS:motorola
-LIBS:texas
-LIBS:intel
-LIBS:audio
-LIBS:interface
-LIBS:digital-audio
-LIBS:philips
-LIBS:display
-LIBS:cypress
-LIBS:siliconi
-LIBS:opto
-LIBS:atmel
-LIBS:contrib
-LIBS:valves
-LIBS:jfng
+EESchema Schematic File Version 4
 LIBS:RPi_Hat-cache
 EELAYER 26 0
@@
 $EndDescr
 $Comp
-L PCA9306-RESCUE-RPi_Hat U6
+L RPi_Hat-rescue:PCA9306-RESCUE-RPi_Hat U6
 U 1 1 58780326
 P 3850 3350
@@
 $EndComp
 $Comp
-L +3.3V #PWR021
+L RPi_Hat-rescue:+3.3V-RESCUE-RPi_Hat #PWR021
 U 1 1 58780337
 P 3175 3000
@@
 $EndComp
 $Comp
-L GND #PWR022
+L RPi_Hat-rescue:GND-RESCUE-RPi_Hat #PWR022
 U 1 1 587A7597
 P 5425 2675
@@
 $EndComp
 $Comp
-L C_Small C13
+L RPi_Hat-rescue:C_Small-RESCUE-RPi_Hat C13
 U 1 1 587A76A7
 P 5275 2550
@@
 $EndComp
 $Comp
-L R R1
+L RPi_Hat-rescue:R-RESCUE-RPi_Hat R1
 U 1 1 587A778D
 P 4550 3000
@@
 	5425 2550 5425 2675
 $Comp
-L GND #PWR023
+L RPi_Hat-rescue:GND-RESCUE-RPi_Hat #PWR023
 U 1 1 5884E7E8
 P 3325 3025
@@
 	3325 3150 3325 3025
 $Comp
-L C C12
+L RPi_Hat-rescue:C-RESCUE-RPi_Hat C12
 U 1 1 58923DFD
 P 6400 3075
@@
 $EndComp
 $Comp
-L C C11
+L RPi_Hat-rescue:C-RESCUE-RPi_Hat C11
 U 1 1 58923E99
 P 6775 3050
@@
 $EndComp
 $Comp
-L GND #PWR024
+L RPi_Hat-rescue:GND-RESCUE-RPi_Hat #PWR024
 U 1 1 5892526A
 P 6600 3275
@@
 	6775 3250 6775 3200
 $Comp
-L DS2482-100 U7
+L jfng:DS2482-100 U7
 U 1 1 5892EED6
 P 5675 3675
@@
 Connection ~ 4975 3975
 $Comp
-L GND #PWR025
+L RPi_Hat-rescue:GND-RESCUE-RPi_Hat #PWR025
 U 1 1 5892FAC8
 P 4975 4075
@@
 $EndComp
 $Comp
-L GND #PWR026
+L RPi_Hat-rescue:GND-RESCUE-RPi_Hat #PWR026
 U 1 1 5892FB06
 P 5675 4500
@@
 	6400 3250 6400 3225
 $Comp
-L +5V #PWR027
+L RPi_Hat-rescue:+5V-RESCUE-RPi_Hat #PWR027
 U 1 1 58930FE6
 P 6600 2725
@@
 Connection ~ 6600 3250
 $Comp
-L GND #PWR028
+L RPi_Hat-rescue:GND-RESCUE-RPi_Hat #PWR028
 U 1 1 589346CB
 P 6650 4075
@@
 	7675 3975 7875 3975
 $Comp
-L DS9503 U8
+L jfng:DS9503 U8
 U 1 1 589346DA
 P 7125 3975
@@
 	4550 2850 4550 2550
 $Comp
-L +5V #PWR029
+L RPi_Hat-rescue:+5V-RESCUE-RPi_Hat #PWR029
 U 1 1 589C5AC0
 P 4700 2425
@@
 _sda
 $Comp
-L R R2
+L RPi_Hat-rescue:R-RESCUE-RPi_Hat R2
 U 1 1 589D4139
 P 4850 3000
@@
 $EndComp
 $Comp
-L R R3
+L RPi_Hat-rescue:R-RESCUE-RPi_Hat R3
 U 1 1 589D4175
 P 5125 3000
