File: Kicad/RPi_GPIO.sch (KiCad schematic (older format))
At the start: 5 parts, among them J1 RPi_GPIO

Commit message: Mise a jour du 6 juillet 2017
Parts:
- D1: value LED -> LED_RED
- D2: value LED -> LED_YELLOW
Other:
- moved on the sheet: D1, R4
Changed lines of the file:
@@
 Thru-Hole Connector
 Wire Wire Line
-	3500 2700 4100 2700
+	3500 2700 3925 2700
+Wire Wire Line
+	3925 2700 4100 2700
 Wire Wire Line
 	3925 2700 3925 2575
 $Comp
-L +3.3V #PWR04
+L +3.3V #PWR05
 U 1 1 5891FB75
 P 3925 2575
-F 0 "#PWR04" H -25 -150 50  0001 C CNN
+F 0 "#PWR05" H -25 -150 50  0001 C CNN
 F 1 "+3.3V" H 3940 2748 50  0000 C CNN
 F 2 "" H -25 0   50  0001 C CNN
@@
 $EndComp
 Wire Wire Line
-	6000 2700 6700 2700
-Wire Wire Line
-	6250 2600 6250 2800
-$Comp
-L +5V #PWR05
+	6000 2700 6250 2700
+Wire Wire Line
+	6250 2700 6700 2700
+Wire Wire Line
+	6250 2600 6250 2700
+Wire Wire Line
+	6250 2700 6250 2800
+$Comp
+L +5V #PWR06
 U 1 1 5891FBCE
 P 6250 2600
-F 0 "#PWR05" H 0   -150 50  0001 C CNN
+F 0 "#PWR06" H 0   -150 50  0001 C CNN
 F 1 "+5V" H 6265 2773 50  0000 C CNN
 F 2 "" H 0   0   50  0001 C CNN
@@
 Connection ~ 6250 2700
 $Comp
-L +3.3V #PWR06
+L +3.3V #PWR07
 U 1 1 5891FC65
 P 3925 3350
-F 0 "#PWR06" H -175 -300 50  0001 C CNN
+F 0 "#PWR07" H -175 -300 50  0001 C CNN
 F 1 "+3.3V" H 3940 3523 50  0000 C CNN
 F 2 "" H -175 -150 50  0001 C CNN
@@
 	3750 3100 3750 3200
 $Comp
-L GND #PWR07
+L GND #PWR08
 U 1 1 5891FD82
 P 3750 3200
-F 0 "#PWR07" H 0   -250 50  0001 C CNN
+F 0 "#PWR08" H 0   -250 50  0001 C CNN
 F 1 "GND" H 3755 3027 50  0000 C CNN
 F 2 "" H 0   0   50  0001 C CNN
@@
 	3750 3900 3750 4000
 $Comp
-L GND #PWR08
+L GND #PWR09
 U 1 1 5891FDD5
 P 3750 4000
-F 0 "#PWR08" H 0   -250 50  0001 C CNN
+F 0 "#PWR09" H 0   -250 50  0001 C CNN
 F 1 "GND" H 3755 3827 50  0000 C CNN
 F 2 "" H 0   0   50  0001 C CNN
@@
 	3750 4600 3750 4675
 $Comp
-L GND #PWR09
+L GND #PWR010
 U 1 1 5891FDFC
 P 3750 4675
-F 0 "#PWR09" H 0   -250 50  0001 C CNN
+F 0 "#PWR010" H 0   -250 50  0001 C CNN
 F 1 "GND" H 3755 4502 50  0000 C CNN
 F 2 "" H 0   0   50  0001 C CNN
@@
 	6350 4300 6350 4375
 $Comp
-L GND #PWR010
+L GND #PWR011
 U 1 1 5891FE4D
 P 6350 4375
-F 0 "#PWR010" H 6400 4425 50  0001 C CNN
+F 0 "#PWR011" H 6400 4425 50  0001 C CNN
 F 1 "GND" H 6450 4275 50  0000 C CNN
 F 2 "" H 0   0   50  0001 C CNN
@@
 	6350 4100 6350 4150
 $Comp
-L GND #PWR011
+L GND #PWR012
 U 1 1 5891FE94
 P 6350 4150
-F 0 "#PWR011" H 6400 4200 50  0001 C CNN
+F 0 "#PWR012" H 6400 4200 50  0001 C CNN
 F 1 "GND" H 6450 4050 50  0000 C CNN
 F 2 "" H 0   0   50  0001 C CNN
@@
 	6900 3600 6900 3675
 $Comp
-L GND #PWR012
+L GND #PWR013
 U 1 1 5891FF6C
 P 6900 3675
-F 0 "#PWR012" H 6950 3725 50  0001 C CNN
+F 0 "#PWR013" H 6950 3725 50  0001 C CNN
 F 1 "GND" H 6975 3550 50  0000 C CNN
 F 2 "" H 550 0   50  0001 C CNN
@@
 	6750 3300 6750 3400
 $Comp
-L GND #PWR013
+L GND #PWR014
 U 1 1 5891FF9A
 P 6750 3400
-F 0 "#PWR013" H 400 -250 50  0001 C CNN
+F 0 "#PWR014" H 400 -250 50  0001 C CNN
 F 1 "GND" H 6850 3275 50  0000 C CNN
 F 2 "" H 400 0   50  0001 C CNN
@@
 $EndComp
 Wire Wire Line
-	6000 2900 6925 2900
+	6000 2900 6775 2900
+Wire Wire Line
+	6775 2900 6925 2900
 Wire Wire Line
 	6775 2900 6775 3000
 $Comp
-L GND #PWR014
+L GND #PWR015
 U 1 1 5892002F
 P 6775 3000
-F 0 "#PWR014" H 425 -250 50  0001 C CNN
+F 0 "#PWR015" H 425 -250 50  0001 C CNN
 F 1 "GND" H 6780 2827 50  0000 C CNN
 F 2 "" H 425 0   50  0001 C CNN
@@
 NoConn ~ 4100 3000
 $Comp
-L PWR_FLAG #FLG015
+L PWR_FLAG #FLG016
 U 1 1 58936B87
 P 3500 2575
-F 0 "#FLG015" H -625 150 50  0001 C CNN
+F 0 "#FLG016" H -625 150 50  0001 C CNN
 F 1 "PWR_FLAG" H 3500 2749 50  0000 C CNN
 F 2 "" H -625 75  50  0001 C CNN
@@
 Connection ~ 3925 2700
 $Comp
-L PWR_FLAG #FLG016
+L PWR_FLAG #FLG017
 U 1 1 58936BD5
 P 6700 2600
-F 0 "#FLG016" H 2575 175 50  0001 C CNN
+F 0 "#FLG017" H 2575 175 50  0001 C CNN
 F 1 "PWR_FLAG" H 6700 2774 50  0000 C CNN
 F 2 "" H 2575 100 50  0001 C CNN
@@
 	6700 2700 6700 2600
 $Comp
-L PWR_FLAG #FLG017
+L PWR_FLAG #FLG018
 U 1 1 58936C10
 P 6925 2825
-F 0 "#FLG017" H 2800 400 50  0001 C CNN
+F 0 "#FLG018" H 2800 400 50  0001 C CNN
 F 1 "PWR_FLAG" H 6925 2999 50  0000 C CNN
 F 2 "" H 2800 325 50  0001 C CNN
@@
 L R R4
 U 1 1 5901649B
-P 3075 4750
-F 0 "R4" H 3155 4750 50  0000 C CNN
-F 1 "1k" V 2975 4750 50  0000 C CNN
-F 2 "Resistors_SMD:R_0805_HandSoldering" V 3005 4750 50  0001 C CNN
-F 3 "" H 3075 4750 50  0000 C CNN
-	1    3075 4750
+P 2875 4750
+F 0 "R4" H 2975 4750 50  0000 C CNN
+F 1 "1k" V 2775 4750 50  0000 C CNN
+F 2 "Resistors_SMD:R_0805_HandSoldering" V 2805 4750 50  0001 C CNN
+F 3 "" H 2875 4750 50  0000 C CNN
+	1    2875 4750
 	1    0    0    -1
 $EndComp
@@
 U 1 1 59016698
 P 3375 4750
-F 0 "R5" H 3455 4750 50  0000 C CNN
+F 0 "R5" H 3475 4750 50  0000 C CNN
 F 1 "1k" V 3275 4750 50  0000 C CNN
 F 2 "Resistors_SMD:R_0805_HandSoldering" V 3305 4750 50  0001 C CNN
@@
 L LED D1
 U 1 1 590167AA
-P 3075 5150
-F 0 "D1" V 3020 5228 50  0000 L CNN
-F 1 "LED" V 3111 5228 50  0000 L CNN
-F 2 "LEDs:LED_0805" H 3075 5150 50  0001 C CNN
-F 3 "" H 3075 5150 50  0001 C CNN
-	1    3075 5150
+P 2875 5150
+F 0 "D1" V 2820 5228 50  0000 L CNN
+F 1 "LED_RED" V 2900 5225 50  0000 L CNN
+F 2 "LEDs:LED_0805" H 2875 5150 50  0001 C CNN
+F 3 "" H 2875 5150 50  0001 C CNN
+	1    2875 5150
 	0    1    1    0
 $EndComp
@@
 P 3375 5150
 F 0 "D2" V 3320 5228 50  0000 L CNN
-F 1 "LED" V 3411 5228 50  0000 L CNN
+F 1 "LED_YELLOW" V 3411 5228 50  0000 L CNN
 F 2 "LEDs:LED_0805" H 3375 5150 50  0001 C CNN
 F 3 "" H 3375 5150 50  0001 C CNN
@@
 $EndComp
 Wire Wire Line
-	4100 4400 3075 4400
-Wire Wire Line
-	3075 4400 3075 4600
+	4100 4400 2875 4400
+Wire Wire Line
+	2875 4400 2875 4600
 Wire Wire Line
 	4100 4500 3375 4500
@@
 	3375 4500 3375 4600
 Wire Wire Line
-	3075 5000 3075 4900
+	2875 5000 2875 4900
 Wire Wire Line
 	3375 5000 3375 4900
 $Comp
-L GND #PWR018
+L GND #PWR019
 U 1 1 59016BFF
-P 3075 5400
-F 0 "#PWR018" H -675 475 50  0001 C CNN
-F 1 "GND" H 3080 5227 50  0000 C CNN
-F 2 "" H -675 725 50  0001 C CNN
-F 3 "" H -675 725 50  0001 C CNN
-	1    3075 5400
-	1    0    0    -1
-$EndComp
-$Comp
-L GND #PWR019
+P 2875 5400
+F 0 "#PWR019" H -875 475 50  0001 C CNN
+F 1 "GND" H 2880 5227 50  0000 C CNN
+F 2 "" H -875 725 50  0001 C CNN
+F 3 "" H -875 725 50  0001 C CNN
+	1    2875 5400
+	1    0    0    -1
+$EndComp
+$Comp
+L GND #PWR020
 U 1 1 59016C14
 P 3375 5400
-F 0 "#PWR019" H -375 475 50  0001 C CNN
+F 0 "#PWR020" H -375 475 50  0001 C CNN
 F 1 "GND" H 3380 5227 50  0000 C CNN
 F 2 "" H -375 725 50  0001 C CNN
@@
 $EndComp
 Wire Wire Line
-	3075 5400 3075 5300
+	2875 5400 2875 5300
 Wire Wire Line
 	3375 5400 3375 5300

Commit message: Reouverture avec une nouvelle version de Kicad
Parts:
- D1, D2: symbol LED -> RPi_Hat-rescue:LED-RESCUE-RPi_Hat
- J1: symbol RPi_GPIO -> jfng:RPi_GPIO
- R4, R5: symbol R -> RPi_Hat-rescue:R-RESCUE-RPi_Hat
Changed lines of the file:
@@
-EESchema Schematic File Version 2
-LIBS:RPi_Hat-rescue
-LIBS:power
-LIBS:device
-LIBS:transistors
-LIBS:conn
-LIBS:linear
-LIBS:regul
-LIBS:74xx
-LIBS:cmos4000
-LIBS:adc-dac
-LIBS:memory
-LIBS:xilinx
-LIBS:microcontrollers
-LIBS:dsp
-LIBS:microchip
-LIBS:analog_switches
-LIBS:motorola
-LIBS:texas
-LIBS:intel
-LIBS:audio
-LIBS:interface
-LIBS:digital-audio
-LIBS:philips
-LIBS:display
-LIBS:cypress
-LIBS:siliconi
-LIBS:opto
-LIBS:atmel
-LIBS:contrib
-LIBS:valves
-LIBS:jfng
+EESchema Schematic File Version 4
 LIBS:RPi_Hat-cache
 EELAYER 26 0
@@
 $EndDescr
 $Comp
-L RPi_GPIO J1
+L jfng:RPi_GPIO J1
 U 1 1 5516AE26
 P 4300 2700
@@
 	3925 2700 3925 2575
 $Comp
-L +3.3V #PWR05
+L RPi_Hat-rescue:+3.3V-RESCUE-RPi_Hat #PWR05
 U 1 1 5891FB75
 P 3925 2575
@@
 	6250 2700 6250 2800
 $Comp
-L +5V #PWR06
+L RPi_Hat-rescue:+5V-RESCUE-RPi_Hat #PWR06
 U 1 1 5891FBCE
 P 6250 2600
@@
 Connection ~ 6250 2700
 $Comp
-L +3.3V #PWR07
+L RPi_Hat-rescue:+3.3V-RESCUE-RPi_Hat #PWR07
 U 1 1 5891FC65
 P 3925 3350
@@
 	3750 3100 3750 3200
 $Comp
-L GND #PWR08
+L RPi_Hat-rescue:GND-RESCUE-RPi_Hat #PWR08
 U 1 1 5891FD82
 P 3750 3200
@@
 	3750 3900 3750 4000
 $Comp
-L GND #PWR09
+L RPi_Hat-rescue:GND-RESCUE-RPi_Hat #PWR09
 U 1 1 5891FDD5
 P 3750 4000
@@
 	3750 4600 3750 4675
 $Comp
-L GND #PWR010
+L RPi_Hat-rescue:GND-RESCUE-RPi_Hat #PWR010
 U 1 1 5891FDFC
 P 3750 4675
@@
 	6350 4300 6350 4375
 $Comp
-L GND #PWR011
+L RPi_Hat-rescue:GND-RESCUE-RPi_Hat #PWR011
 U 1 1 5891FE4D
 P 6350 4375
@@
 	6350 4100 6350 4150
 $Comp
-L GND #PWR012
+L RPi_Hat-rescue:GND-RESCUE-RPi_Hat #PWR012
 U 1 1 5891FE94
 P 6350 4150
@@
 	6900 3600 6900 3675
 $Comp
-L GND #PWR013
+L RPi_Hat-rescue:GND-RESCUE-RPi_Hat #PWR013
 U 1 1 5891FF6C
 P 6900 3675
@@
 	6750 3300 6750 3400
 $Comp
-L GND #PWR014
+L RPi_Hat-rescue:GND-RESCUE-RPi_Hat #PWR014
 U 1 1 5891FF9A
 P 6750 3400
@@
 	6775 2900 6775 3000
 $Comp
-L GND #PWR015
+L RPi_Hat-rescue:GND-RESCUE-RPi_Hat #PWR015
 U 1 1 5892002F
 P 6775 3000
@@
 NoConn ~ 4100 3000
 $Comp
-L PWR_FLAG #FLG016
+L RPi_Hat-rescue:PWR_FLAG-RESCUE-RPi_Hat #FLG016
 U 1 1 58936B87
 P 3500 2575
@@
 Connection ~ 3925 2700
 $Comp
-L PWR_FLAG #FLG017
+L RPi_Hat-rescue:PWR_FLAG-RESCUE-RPi_Hat #FLG017
 U 1 1 58936BD5
 P 6700 2600
@@
 	6700 2700 6700 2600
 $Comp
-L PWR_FLAG #FLG018
+L RPi_Hat-rescue:PWR_FLAG-RESCUE-RPi_Hat #FLG018
 U 1 1 58936C10
 P 6925 2825
@@
 RPi_CLK_SPI
 $Comp
-L R R4
+L RPi_Hat-rescue:R-RESCUE-RPi_Hat R4
 U 1 1 5901649B
 P 2875 4750
@@
 $EndComp
 $Comp
-L R R5
+L RPi_Hat-rescue:R-RESCUE-RPi_Hat R5
 U 1 1 59016698
 P 3375 4750
@@
 $EndComp
 $Comp
-L LED D1
+L RPi_Hat-rescue:LED-RESCUE-RPi_Hat D1
 U 1 1 590167AA
 P 2875 5150
@@
 $EndComp
 $Comp
-L LED D2
+L RPi_Hat-rescue:LED-RESCUE-RPi_Hat D2
 U 1 1 59016879
 P 3375 5150
@@
 	3375 5000 3375 4900
 $Comp
-L GND #PWR019
+L RPi_Hat-rescue:GND-RESCUE-RPi_Hat #PWR019
 U 1 1 59016BFF
 P 2875 5400
@@
 $EndComp
 $Comp
-L GND #PWR020
+L RPi_Hat-rescue:GND-RESCUE-RPi_Hat #PWR020
 U 1 1 59016C14
 P 3375 5400
