File: Kicad/RTC.sch (KiCad schematic (older format))
At the start: 3 parts, among them U1 DS3231

Commit message: Mise a jour du 6 juillet 2017
Connections:
- net INT_SQW: now reaches U1.3 (~INT~/SQW)
- no-connect marks 3 -> 2
Changed lines of the file:
@@
 $Descr USLetter 11000 8500
 encoding utf-8
-Sheet 3 7
+Sheet 6 7
 Title ""
 Date "2017-02-08"
@@
 $EndComp
 $Comp
-L GND #PWR020
+L GND #PWR048
 U 1 1 587B605B
 P 4675 3275
-F 0 "#PWR020" H 4675 3025 50  0001 C CNN
+F 0 "#PWR048" H 4675 3025 50  0001 C CNN
 F 1 "GND" H 4675 3125 50  0000 C CNN
 F 2 "" H 4675 3275 50  0000 C CNN
@@
 	4675 3175 4675 3275
 $Comp
-L +3.3V #PWR021
+L +3.3V #PWR049
 U 1 1 587B639C
 P 4675 1875
-F 0 "#PWR021" H 4675 1725 50  0001 C CNN
+F 0 "#PWR049" H 4675 1725 50  0001 C CNN
 F 1 "+3.3V" H 4675 2015 50  0000 C CNN
 F 2 "" H 4675 1875 50  0000 C CNN
@@
 NoConn ~ 4175 2875
 NoConn ~ 5175 2675
-NoConn ~ 5175 2575
 $Comp
 L Battery_Cell BT1
@@
 $EndComp
 Wire Wire Line
-	5175 2875 5625 2875
+	5175 2875 6050 2875
 Wire Wire Line
 	5450 3175 5450 3225
@@
 Connection ~ 4675 3225
 $Comp
-L PWR_FLAG #FLG022
+L PWR_FLAG #FLG050
 U 1 1 589372D2
-P 5625 2800
-F 0 "#FLG022" H -75 175 50  0001 C CNN
-F 1 "PWR_FLAG" H 5625 2974 50  0000 C CNN
-F 2 "" H -75 100 50  0001 C CNN
-F 3 "" H -75 100 50  0001 C CNN
-	1    5625 2800
+P 6050 2800
+F 0 "#FLG050" H 350 175 50  0001 C CNN
+F 1 "PWR_FLAG" H 6050 2974 50  0000 C CNN
+F 2 "" H 350 100 50  0001 C CNN
+F 3 "" H 350 100 50  0001 C CNN
+	1    6050 2800
 	1    0    0    -1
 $EndComp
 Wire Wire Line
-	5625 2875 5625 2800
+	6050 2875 6050 2800
 Connection ~ 5450 2875
 Text HLabel 4175 2575 0    60   Input ~ 0
@@
 Connection ~ 4675 1925
 $Comp
-L GND #PWR023
+L GND #PWR051
 U 1 1 589C27AC
 P 5625 2275
-F 0 "#PWR023" H 475 -275 50  0001 C CNN
+F 0 "#PWR051" H 475 -275 50  0001 C CNN
 F 1 "GND" H 5630 2102 50  0000 C CNN
 F 2 "" H 475 -25 50  0001 C CNN
@@
 Text Label 5200 2875 0    60   ~ 0
 VBAT
+Text HLabel 5175 2575 2    60   Output ~ 0
+INT_SQW
 $EndSCHEMATC

Commit message: Reouverture avec une nouvelle version de Kicad
Parts:
- BT1: symbol Battery_Cell -> RPi_Hat-rescue:Battery_Cell-RESCUE-RPi_Hat
- C14: symbol C_Small -> RPi_Hat-rescue:C_Small-RESCUE-RPi_Hat
- U1: symbol DS3231 -> jfng:DS3231
Changed lines of the file:
@@
-EESchema Schematic File Version 2
-LIBS:RPi_Hat-rescue
-LIBS:power
-LIBS:device
-LIBS:transistors
-LIBS:conn
-LIBS:linear
-LIBS:regul
-LIBS:74xx
-LIBS:cmos4000
-LIBS:adc-dac
-LIBS:memory
-LIBS:xilinx
-LIBS:microcontrollers
-LIBS:dsp
-LIBS:microchip
-LIBS:analog_switches
-LIBS:motorola
-LIBS:texas
-LIBS:intel
-LIBS:audio
-LIBS:interface
-LIBS:digital-audio
-LIBS:philips
-LIBS:display
-LIBS:cypress
-LIBS:siliconi
-LIBS:opto
-LIBS:atmel
-LIBS:contrib
-LIBS:valves
-LIBS:jfng
+EESchema Schematic File Version 4
 LIBS:RPi_Hat-cache
 EELAYER 26 0
@@
 $EndDescr
 $Comp
-L DS3231 U1
+L jfng:DS3231 U1
 U 1 1 587B5F3E
 P 4675 2675
@@
 $EndComp
 $Comp
-L GND #PWR048
+L RPi_Hat-rescue:GND-RESCUE-RPi_Hat #PWR048
 U 1 1 587B605B
 P 4675 3275
@@
 	4675 3175 4675 3275
 $Comp
-L +3.3V #PWR049
+L RPi_Hat-rescue:+3.3V-RESCUE-RPi_Hat #PWR049
 U 1 1 587B639C
 P 4675 1875
@@
 NoConn ~ 5175 2675
 $Comp
-L Battery_Cell BT1
+L RPi_Hat-rescue:Battery_Cell-RESCUE-RPi_Hat BT1
 U 1 1 587B6407
 P 5450 3075
@@
 Connection ~ 4675 3225
 $Comp
-L PWR_FLAG #FLG050
+L RPi_Hat-rescue:PWR_FLAG-RESCUE-RPi_Hat #FLG050
 U 1 1 589372D2
 P 6050 2800
@@
 SDA
 $Comp
-L C_Small C14
+L RPi_Hat-rescue:C_Small-RESCUE-RPi_Hat C14
 U 1 1 589C24D4
 P 5625 2025
@@
 Connection ~ 4675 1925
 $Comp
-L GND #PWR051
+L RPi_Hat-rescue:GND-RESCUE-RPi_Hat #PWR051
 U 1 1 589C27AC
 P 5625 2275
